File: KiCadProjects/synth_psu/synth_psu.kicad_sch (KiCad schematic)
At the start: 27 parts, among them J1 Barrel_Jack, J2 Switch Terminals, J3 Output Terminals, J4 Fan 1, J5 Fan 2, U1 LM7815_TO220, U2 LM7915_TO220

Commit message: remove old projects
Parts:
- C1, C2, C3, C4, C5, C6: Link (none) -> https://www.digikey.com/en/products/detail/rubycon/50PK4700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; Part No. (none) -> 1189-1397-ND
- C10, C7, C8, C9: Link (none) -> https://www.digikey.com/en/products/detail/kemet/C330C105K5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; Part No. (none) -> 399-9886-1-ND
- D1, D2, D3: Link (none) -> https://www.digikey.com/en/products/detail/diotec-semicondu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; Part No. (none) -> 4878-1N4007CT-ND
- D4, D5: Link (none) -> https://www.digikey.com/en/products/detail/w%C3%BCrth-elekt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; Part No. (none) -> 732-5016-ND
- F1: Link (none) -> https://www.digikey.com/en/products/detail/littelfuse-inc/0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; Part No. (none) -> F6094-ND
- J2: Link (none) -> https://www.digikey.com/en/products/detail/te-connectivity-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; Part No. (none) -> A98333-ND
- J3: Link (none) -> https://www.digikey.com/en/products/detail/te-connectivity-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; Part No. (none) -> A98334-ND
- J4, J5: Link (none) -> https://www.digikey.com/en/products/detail/harwin-inc/M20-9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; Part No. (none) -> 952-2262-ND
- L1, L2: Link (none) -> https://www.digikey.com/en/products/detail/bourns-inc/2124-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; Part No. (none) -> M8863-ND
- R1, R2: value 330 -> 1k; Link (none) -> https://www.digikey.com/en/products/detail/stackpole-electr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; Part No. (none) -> CF12JT1K00CT-ND
- U1: Link (none) -> https://www.digikey.com/en/products/detail/texas-instrument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; Part No. (none) -> 296-44418-5-ND
- U2: Link (none) -> https://www.digikey.com/en/products/detail/texas-instrument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; Part No. (none) -> LM7915CT/NOPB-ND
