File: KiCadProjects/vco/vco.kicad_sch (KiCad schematic)
At the start: 0 parts

Commit message: updating github
Parts:
- added C1, C4, C7: 2.2nF, symbol Device:C
- added C2, C3, C5, C6, C8, C9: 1uF, symbol Device:C
- added D1, D2, D3, D4, D5, D6: 1N4148, Diode_THT:D_DO-35_SOD27_P7.62mm_Horizontal, symbol Diode:1N4148
- added Q1, Q4, Q6: BC548, Package_TO_SOT_THT:TO-92_Inline, symbol Transistor_BJT:BC548
- added Q2, Q3, Q5: BC558, Package_TO_SOT_THT:TO-92_Inline, symbol Transistor_BJT:BC558
- added R1, R16, R19, R30, R33, R4: 1M, symbol Device:R_US
- added R10, R12, R14, R17, R20, R23, R24, R26, R28, R31, R34, R37, R38, R40, R42, R5, R6, R8: 100k, symbol Device:R_US
- added R11, R13, R25, R27, R39, R41: 20k, symbol Device:R_US
- added R15, R29, R3: 100K, symbol Device:R_US
- added R18, R2, R32: 1.5k, symbol Device:R_US
- added R21, R35, R7: 200k, symbol Device:R_US
- added R22, R36, R9: 33k, symbol Device:R_US
- added RV1, RV11, RV7: 1k, symbol Device:R_Potentiometer_Trim_US
- added RV10, RV12, RV2, RV3, RV4, RV5, RV6, RV8, RV9: 100k, symbol Device:R_Potentiometer_US
- added TH1, TH2, TH3, TH4, TH5, TH6, TH7, TH8, TH9: 10k, symbol Device:Thermistor_NTC_US
- added U1: 40106, symbol 4xxx:40106
- added U2, U3, U4: TL074, symbol Amplifier_Operational:TL074
Connections:
- new net: D2.1 (K), R8.1, U1.3
- new net: C3.1, U1.4
- new net: R22.1, R24.1, U3.9 (-)
- new net: R17.2, TH6.1
- new net: Q3.2 (B), R18.1, TH4.2, TH5.2, TH6.2
- new net: R30.1, RV10.2
- new net: R30.2, TH8.1
- new net: C1.1, D1.1 (K), Q1.1 (C), U1.1, U2.3 (+)
- new net: D6.1 (K), R37.1, U1.13
- new net: D6.2 (A), R35.1, U4.7
- new net: R35.2, RV12.1, U4.6 (-)
- new net: C6.1, U1.8
- new net: D4.1 (K), R23.1, U1.9
- new net: R38.2, R39.1, U4.8
- new net: D1.2 (A), U1.2
- new net: C5.2, R20.1, U3.10 (+), U3.5 (+)
- new net: R21.2, RV8.1, U3.6 (-)
- new net: D4.2 (A), R21.1, U3.7
- new net: R24.2, R25.1, U3.8
- new net: R16.1, RV6.2
- new net: C5.1, U3.1, U3.2 (-)
- new net: C8.2, R34.1, U4.10 (+), U4.5 (+)
- new net: R36.1, R38.1, U4.9 (-)
- new net: C4.1, D3.1 (K), Q4.1 (C), U1.5, U3.3 (+)
- new net: D3.2 (A), U1.6
- new net: R10.1, R9.1, U2.9 (-)
- new net: R10.2, R11.1, U2.8
- new net: R18.2, RV7.1
- new net: Q3.3 (E), Q4.2 (B), R19.2
- new net: R3.2, RV2.2
- new net: C3.2, R12.1, R13.1
- new net: C6.2, R26.1, R27.1
- new net: R3.1, TH1.1
- new net: R16.2, TH5.1
- new net: D2.2 (A), R7.1, U2.7
- new net: R7.2, RV4.1, U2.6 (-)
- new net: C2.2, R6.1, U2.10 (+), U2.5 (+)
- new net: Q5.2 (B), R32.1, TH7.2, TH8.2, TH9.2
- new net: R32.2, RV11.1
- new net: R15.2, RV5.2
- new net: C9.1, U1.12
- new net: Q5.3 (E), Q6.2 (B), R33.2
- new net: C7.1, D5.1 (K), Q6.1 (C), U1.11, U4.3 (+)
- new net: D5.2 (A), U1.10
- new net: C9.2, R40.1, R41.1
- new net: Q2.2 (B), R2.1, TH1.2, TH2.2, TH3.2
- new net: Q1.2 (B), Q2.3 (E), R1.2
- new net: R15.1, TH4.1
- new net: R2.2, RV1.1
- new net: R4.2, TH2.1
- new net: R29.2, RV9.2
- new net: R4.1, RV3.2
- new net: R5.2, TH3.1
- new net: C8.1, U4.1, U4.2 (-)
- new net: R31.2, TH9.1
- new net: R29.1, TH7.1
- new net: C2.1, U2.1, U2.2 (-)
- new net +15V: R1.1, R19.1, R33.1
- new net -15V: Q2.1 (C), Q3.1 (C), Q5.1 (C), RV10.3, RV2.3, RV3.3, RV5.3, RV6.3, RV9.3
- new net CV1: R5.1
- new net CV2: R17.1
- new net CV3: R31.1
- new net GND: C1.2, C4.2, C7.2, Q1.3 (E), Q4.3 (E), Q6.3 (E), R12.2, R14.2, R20.2, R22.2, R23.2, R26.2, R28.2, R34.2, R36.2, R37.2, R40.2, R42.2, R6.2, R8.2, R9.2, RV1.2, RV1.3, RV10.1, RV11.2, RV11.3, RV12.2, RV12.3, RV2.1, RV3.1, RV4.2, RV4.3, RV5.1, RV6.1, RV7.2, RV7.3, RV8.2, RV8.3, RV9.1
- new net SAW1: R11.2
- new net SAW2: R25.2
- new net SAW3: R39.2
- new net SQ1: R13.2, R14.1
- new net SQ2: R27.2, R28.1
- new net SQ3: R41.2, R42.1
Other:
- note added: "Coarse"
- note added: "Fine"

Commit message: vco updates
Parts:
- U1, U2, U3, U4: footprint (none) -> Package_DIP:DIP-14_W7.62mm_Socket
Changed lines of the file:
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@@
 			)
 		)
-		(property "Footprint" ""
+		(property "Footprint" "Package_DIP:DIP-14_W7.62mm_Socket"
 			(at 157.48 52.07 0)
 			(effects
@@
 			)
 		)
-		(property "Footprint" ""
+		(property "Footprint" "Package_DIP:DIP-14_W7.62mm_Socket"
 			(at 158.75 138.43 0)
 			(effects
@@
 			)
 		)
-		(property "Footprint" ""
+		(property "Footprint" "Package_DIP:DIP-14_W7.62mm_Socket"
 			(at 111.76 81.28 0)
 			(effects
@@
 			)
 		)
-		(property "Footprint" ""
+		(property "Footprint" "Package_DIP:DIP-14_W7.62mm_Socket"
 			(at 114.3 135.89 0)
 			(effects
@@
 			)
 		)
-		(property "Footprint" ""
+		(property "Footprint" "Package_DIP:DIP-14_W7.62mm_Socket"
 			(at 143.51 111.76 0)
 			(effects
@@
 			)
 		)
-		(property "Footprint" ""
+		(property "Footprint" "Package_DIP:DIP-14_W7.62mm_Socket"
 			(at 356.87 49.53 0)
 			(effects
@@
 			)
 		)
-		(property "Footprint" ""
+		(property "Footprint" "Package_DIP:DIP-14_W7.62mm_Socket"
 			(at 142.24 198.12 0)
 			(effects
@@
 			)
 		)
-		(property "Footprint" ""
+		(property "Footprint" "Package_DIP:DIP-14_W7.62mm_Socket"
 			(at 113.03 167.64 0)
 			(effects
@@
 			)
 		)
-		(property "Footprint" ""
+		(property "Footprint" "Package_DIP:DIP-14_W7.62mm_Socket"
 			(at 401.32 135.89 0)
 			(effects
@@
 			)
 		)
-		(property "Footprint" ""
+		(property "Footprint" "Package_DIP:DIP-14_W7.62mm_Socket"
 			(at 384.81 137.16 0)
 			(effects
@@
 			)
 		)
-		(property "Footprint" ""
+		(property "Footprint" "Package_DIP:DIP-14_W7.62mm_Socket"
 			(at 142.24 25.4 0)
 			(effects
@@
 			)
 		)
-		(property "Footprint" ""
+		(property "Footprint" "Package_DIP:DIP-14_W7.62mm_Socket"
 			(at 401.32 152.4 0)
 			(effects
@@
 			)
 		)
-		(property "Footprint" ""
+		(property "Footprint" "Package_DIP:DIP-14_W7.62mm_Socket"
 			(at 157.48 224.79 0)
 			(effects
@@
 			)
 		)
-		(property "Footprint" ""
+		(property "Footprint" "Package_DIP:DIP-14_W7.62mm_Socket"
 			(at 384.81 153.67 0)
 			(effects
@@
 			)
 		)
-		(property "Footprint" ""
+		(property "Footprint" "Package_DIP:DIP-14_W7.62mm_Socket"
 			(at 340.36 50.8 0)
 			(effects
@@
 			)
 		)
-		(property "Footprint" ""
+		(property "Footprint" "Package_DIP:DIP-14_W7.62mm_Socket"
 			(at 109.22 109.22 0)
 			(effects
@@
 			)
 		)
-		(property "Footprint" ""
+		(property "Footprint" "Package_DIP:DIP-14_W7.62mm_Socket"
 			(at 107.95 195.58 0)
 			(effects
@@
 			)
 		)
-		(property "Footprint" ""
+		(property "Footprint" "Package_DIP:DIP-14_W7.62mm_Socket"
 			(at 111.76 254 0)
 			(effects
@@
 			)
 		)
-		(property "Footprint" ""
+		(property "Footprint" "Package_DIP:DIP-14_W7.62mm_Socket"
 			(at 113.03 222.25 0)
 			(effects
@@
 			)
 		)
-		(property "Footprint" ""
+		(property "Footprint" "Package_DIP:DIP-14_W7.62mm_Socket"
 			(at 113.03 49.53 0)
 			(effects
@@
 			)
 		)
-		(property "Footprint" ""
+		(property "Footprint" "Package_DIP:DIP-14_W7.62mm_Socket"
 			(at 107.95 22.86 0)
 			(effects
@@
 			)
 		)
-		(property "Footprint" ""
+		(property "Footprint" "Package_DIP:DIP-14_W7.62mm_Socket"
 			(at 368.3 44.45 0)
 			(effects
